Commit message: [fix]：修复对称性损失缺失时的报错；

File: resources/robots/biped_s45/urdf/biped_s45.urdf (robot description, URDF)
Before this commit: robot biped_s45, 47 links, 46 joints
Links:
- link leg_l6_link: geometry collision mesh filename=../meshes/l_foot_roll.STL; visual mesh filename=../meshes/l_foot_roll.STL
- link leg_r6_link: geometry collision mesh filename=../meshes/r_foot_roll.STL; visual mesh filename=../meshes/r_foot_roll.STL
