Commit message: [feat]:惩罚机器人脚步岔开走路的姿态，补充行走时的相位，增加动作幅度惩罚

File: resources/robots/biped_s45/urdf/biped_s45_waist_cam.urdf (robot description, URDF)
Before this commit: robot biped_s45, 53 links, 52 joints
Joints:
- joint waist_camera: origin xyz=0.168717483101422 0 0.01355599662743 rpy=0 0 0 -> xyz=0.168717483101422 0 0.01355599662743 rpy=0 0.698  0
